Commit message: adding blinker control and comments solving some bugs TODO: refactor in typescript

File: scooter_javascript/demo1/urdf-loaders/urdf/thormang3/urdf/all.urdf (robot description, URDF)
Before this commit: robot gogoro_and_thormang3, 49 links, 48 joints
Links:
- added link blinker_left, mass 0.01; collision box size=0.05 0.09 0.085; visual box size=0.05 0.09 0.085
- added link blinker_right, mass 0.01; collision box size=0.05 0.09 0.085; visual box size=0.05 0.09 0.085
- added link stop_light, mass 0.01; collision box size=0.05 0.26 0.085; visual box size=0.05 0.26 0.085
Joints:
- added joint rigid1: type fixed, parent body, child stop_light, origin xyz=-0.52 0 0.67 rpy=0 0 0
- added joint rigid2: type fixed, parent body, child blinker_left, origin xyz=-0.49 0.15 0.67 rpy=0 0 0
- added joint rigid3: type fixed, parent body, child blinker_right, origin xyz=-0.49 -0.15 0.67 rpy=0 0 0
