Commit message: changing the controls and adding orientation check

File: scooter_javascript/demo1/urdf-loaders/urdf/track/urdf/model.urdf (robot description, URDF)
Before this commit: robot track, 33 links, 32 joints
Links:
- added link pylon_1, mass 1.0; collision mesh filename=../meshes/pylons/pylon.stl scale=4 4 4; visual mesh filename=../meshes/pylons/pylon.stl scale=4 4 4
- added link pylon_10, mass 1.0; collision mesh filename=../meshes/pylons/pylon.stl scale=4 4 4; visual mesh filename=../meshes/pylons/pylon.stl scale=4 4 4
- added link pylon_11, mass 1.0; collision mesh filename=../meshes/pylons/pylon.stl scale=4 4 4; visual mesh filename=../meshes/pylons/pylon.stl scale=4 4 4
- added link pylon_12, mass 1.0; collision mesh filename=../meshes/pylons/pylon.stl scale=4 4 4; visual mesh filename=../meshes/pylons/pylon.stl scale=4 4 4
- added link pylon_13, mass 1.0; collision mesh filename=../meshes/pylons/pylon.stl scale=4 4 4; visual mesh filename=../meshes/pylons/pylon.stl scale=4 4 4
- added link pylon_2, mass 1.0; collision mesh filename=../meshes/pylons/pylon.stl scale=4 4 4; visual mesh filename=../meshes/pylons/pylon.stl scale=4 4 4
- added link pylon_3, mass 1.0; collision mesh filename=../meshes/pylons/pylon.stl scale=4 4 4; visual mesh filename=../meshes/pylons/pylon.stl scale=4 4 4
- added link pylon_4, mass 1.0; collision mesh filename=../meshes/pylons/pylon.stl scale=4 4 4; visual mesh filename=../meshes/pylons/pylon.stl scale=4 4 4
- added link pylon_5, mass 1.0; collision mesh filename=../meshes/pylons/pylon.stl scale=4 4 4; visual mesh filename=../meshes/pylons/pylon.stl scale=4 4 4
- added link pylon_6, mass 1.0; collision mesh filename=../meshes/pylons/pylon.stl scale=4 4 4; visual mesh filename=../meshes/pylons/pylon.stl scale=4 4 4
- added link pylon_7, mass 1.0; collision mesh filename=../meshes/pylons/pylon.stl scale=4 4 4; visual mesh filename=../meshes/pylons/pylon.stl scale=4 4 4
- added link pylon_8, mass 1.0; collision mesh filename=../meshes/pylons/pylon.stl scale=4 4 4; visual mesh filename=../meshes/pylons/pylon.stl scale=4 4 4
- added link pylon_9, mass 1.0; collision mesh filename=../meshes/pylons/pylon.stl scale=4 4 4; visual mesh filename=../meshes/pylons/pylon.stl scale=4 4 4
- link base_1_train: geometry collision mesh filename=../meshes/train_cross_light/base_1.stl scale=0.002 0.002 0.002; visual mesh filename=../meshes/train_cross_light/base_1.stl scale=0.002 0.002 0.002
- link base_link_traffic: geometry collision mesh filename=../meshes/traffic_light/base_link.stl scale=0.002 0.002 0.002; visual mesh filename=../meshes/traffic_light/base_link.stl scale=0.002 0.002 0.002
- link body_1: geometry collision mesh filename=../meshes/zebra_light/zebra_body.stl scale=0.002 0.002 0.002; visual mesh filename=../meshes/zebra_light/zebra_body.stl scale=0.002 0.002 0.002
- link body_1_traffic: geometry collision mesh filename=../meshes/traffic_light/body_1.stl scale=0.002 0.002 0.002; visual mesh filename=../meshes/traffic_light/body_1.stl scale=0.002 0.002 0.002
- link green_1_traffic: geometry collision mesh filename=../meshes/traffic_light/green_1.stl scale=0.002 0.002 0.002; visual mesh filename=../meshes/traffic_light/green_1.stl scale=0.002 0.002 0.002
- link left_1: geometry collision mesh filename=../meshes/zebra_light/left_1.stl scale=0.002 0.002 0.002; visual mesh filename=../meshes/zebra_light/left_1.stl scale=0.002 0.002 0.002
- link left_1_train: geometry collision mesh filename=../meshes/train_cross_light/left_1.stl scale=0.002 0.002 0.002; visual mesh filename=../meshes/train_cross_light/left_1.stl scale=0.002 0.002 0.002
- link red_1_traffic: geometry collision mesh filename=../meshes/traffic_light/red_1.stl scale=0.002 0.002 0.002; visual mesh filename=../meshes/traffic_light/red_1.stl scale=0.002 0.002 0.002
- link right_1: geometry collision mesh filename=../meshes/zebra_light/right_1.stl scale=0.002 0.002 0.002; visual mesh filename=../meshes/zebra_light/right_1.stl scale=0.002 0.002 0.002
- link right_1_train: geometry collision mesh filename=../meshes/train_cross_light/right_1.stl scale=0.002 0.002 0.002; visual mesh filename=../meshes/train_cross_light/right_1.stl scale=0.002 0.002 0.002
- link yellow_1_traffic: geometry collision mesh filename=../meshes/traffic_light/yellow_1.stl scale=0.002 0.002 0.002; visual mesh filename=../meshes/traffic_light/yellow_1.stl scale=0.002 0.002 0.002
Joints:
- added joint Rigid1_pylon1: type fixed, parent world, child pylon_1, origin xyz=-13.25 -16.3 0 rpy=0 0 2.5
- added joint Rigid1_pylon10: type fixed, parent world, child pylon_10, origin xyz=4.7 -20.7 0 rpy=0 0 3.14
- added joint Rigid1_pylon11: type fixed, parent world, child pylon_11, origin xyz=6.1 -20 0 rpy=0 0 4.7
- added joint Rigid1_pylon12: type fixed, parent world, child pylon_12, origin xyz=6.1 -17.9 0 rpy=0 0 4.7
- added joint Rigid1_pylon13: type fixed, parent world, child pylon_13, origin xyz=6.1 -15.8 0 rpy=0 0 4.7
- added joint Rigid1_pylon2: type fixed, parent world, child pylon_2, origin xyz=-11.5 -17.3 0 rpy=0 0 2.7
- added joint Rigid1_pylon3: type fixed, parent world, child pylon_3, origin xyz=-9.5 -17.9 0 rpy=0 0 3.0
- added joint Rigid1_pylon4: type fixed, parent world, child pylon_4, origin xyz=-7.4 -18 0 rpy=0 0 3.14
- added joint Rigid1_pylon5: type fixed, parent world, child pylon_5, origin xyz=-5.4 -18.5 0 rpy=0 0 2.7
- added joint Rigid1_pylon6: type fixed, parent world, child pylon_6, origin xyz=-3.5 -19.4 0 rpy=0 0 2.7
- added joint Rigid1_pylon7: type fixed, parent world, child pylon_7, origin xyz=-1.6 -20.3 0 rpy=0 0 2.7
- added joint Rigid1_pylon8: type fixed, parent world, child pylon_8, origin xyz=0.35 -20.7 0 rpy=0 0 3.14
- added joint Rigid1_pylon9: type fixed, parent world, child pylon_9, origin xyz=2.5 -20.7 0 rpy=0 0 3.14
- joint Rigid1_traffic: origin xyz=7 -17 0.75 rpy=1.57 0 3.14 -> xyz=7 -17 1.5 rpy=1.57 0 3.14
- joint Rigid2_traffic: origin xyz=7 -17 0.75 rpy=1.57 0 3.14 -> xyz=7 -17 1.5 rpy=1.57 0 3.14
- joint Rigid3_traffic: origin xyz=7 -17 0.75 rpy=1.57 0 3.14  -> xyz=7 -17 1.5 rpy=1.57 0 3.14 
- joint Rigid4_traffic: origin xyz=7 -17 0.75 rpy=1.57 0 3.14 -> xyz=7 -17 1.5 rpy=1.57 0 3.14
- joint Rigid4_zebra: origin xyz=-13.505 -15 1 rpy=1.57 0 1.57 -> xyz=-13.505 -15 2 rpy=1.57 0 1.57
- joint Rigid5_traffic: origin xyz=7 -17 0.75 rpy=1.57 0 3.14 -> xyz=7 -17 1.5 rpy=1.57 0 3.14
- joint Rigid5_zebra: origin xyz=-13.565 -15.005 0.875 rpy=0 0 1.57 -> xyz=-13.625 -15.005 1.75 rpy=0 0 1.57
- joint Rigid6_zebra: origin xyz=-13.415 -15.005 0.72 rpy=0 0 1.57 -> xyz=-13.325 -15.005 1.44 rpy=0 0 1.57

Commit message: adding the textures for the pylons

File: scooter_javascript/demo1/urdf-loaders/urdf/track/urdf/model.urdf (robot description, URDF)
Before this commit: robot track, 46 links, 45 joints
Links:
- link pylon_1: geometry collision mesh filename=../meshes/pylons/test_pylon.dae scale=4 4 4; visual mesh filename=../meshes/pylons/test_pylon.dae scale=4 4 4
- link pylon_10: geometry collision mesh filename=../meshes/pylons/test_pylon.dae scale=4 4 4; visual mesh filename=../meshes/pylons/test_pylon.dae scale=4 4 4
- link pylon_11: geometry collision mesh filename=../meshes/pylons/test_pylon.dae scale=4 4 4; visual mesh filename=../meshes/pylons/test_pylon.dae scale=4 4 4
- link pylon_12: geometry collision mesh filename=../meshes/pylons/test_pylon.dae scale=4 4 4; visual mesh filename=../meshes/pylons/test_pylon.dae scale=4 4 4
- link pylon_13: geometry collision mesh filename=../meshes/pylons/test_pylon.dae scale=4 4 4; visual mesh filename=../meshes/pylons/test_pylon.dae scale=4 4 4
- link pylon_2: geometry collision mesh filename=../meshes/pylons/test_pylon.dae scale=4 4 4; visual mesh filename=../meshes/pylons/test_pylon.dae scale=4 4 4
- link pylon_3: geometry collision mesh filename=../meshes/pylons/test_pylon.dae scale=4 4 4; visual mesh filename=../meshes/pylons/test_pylon.dae scale=4 4 4
- link pylon_4: geometry collision mesh filename=../meshes/pylons/test_pylon.dae scale=4 4 4; visual mesh filename=../meshes/pylons/test_pylon.dae scale=4 4 4
- link pylon_5: geometry collision mesh filename=../meshes/pylons/test_pylon.dae scale=4 4 4; visual mesh filename=../meshes/pylons/test_pylon.dae scale=4 4 4
- link pylon_6: geometry collision mesh filename=../meshes/pylons/test_pylon.dae scale=4 4 4; visual mesh filename=../meshes/pylons/test_pylon.dae scale=4 4 4
- link pylon_7: geometry collision mesh filename=../meshes/pylons/test_pylon.dae scale=4 4 4; visual mesh filename=../meshes/pylons/test_pylon.dae scale=4 4 4
- link pylon_8: geometry collision mesh filename=../meshes/pylons/test_pylon.dae scale=4 4 4; visual mesh filename=../meshes/pylons/test_pylon.dae scale=4 4 4
- link pylon_9: geometry collision mesh filename=../meshes/pylons/test_pylon.dae scale=4 4 4; visual mesh filename=../meshes/pylons/test_pylon.dae scale=4 4 4
