Commit message: adding the forward kin to the robot

File: assets/urdf/thormang3/urdf/all.urdf (robot description, URDF)
Before this commit: robot gogoro_and_thormang3, 52 links, 51 joints
Links:
- removed link root_link
- added link dumy
- added link feet_visual, mass 0.01; visual box size=0.15 0.1 0.1
- added link scooter_grip_L, mass 0.001; visual box size=0.001 0.001 0.001
- added link scooter_grip_R, mass 0.001; visual box size=0.001 0.001 0.001
Joints:
- removed joint rigid1
- removed joint root_joint
- added joint rigid01: type fixed, parent dumy, child pelvis_link, origin xyz=0.0 0.0 0.0 rpy=-1.57079632679 0 0
- added joint rigid02: type fixed, parent body, child stop_light, origin xyz=-0.52 0 0.67 rpy=0 0 0
- added joint rigid100: type fixed, parent head, child scooter_grip_L, origin xyz=0.0 0.25 0.25 rpy=0 0 0
- added joint rigid101: type fixed, parent head, child scooter_grip_R, origin xyz=0.0 -0.25 0.25 rpy=0 0 0
- added joint rigid4: type revolute, parent body, child feet_visual, origin xyz=0.0 -0.2 0.0 rpy=0 0 0, limit lower=0 upper=0 effort=1000 velocity=6.5
- joint cam: origin xyz=0.0682 0.045 0.056 rpy=0 0 0 -> xyz=0.0682 0.045 0.056 rpy=-1.570796327 0 -1.570796327
- joint l_arm_el_y: limit lower=-1.2566370616 upper=1.2566370616 effort=1000 velocity=6.5 -> lower=-1.570796327 upper=1.570796327 effort=1000 velocity=6.5
- joint l_arm_end: axis (none) -> 0 1 0; limit (none) -> lower=0 upper=0 effort=1000000 velocity=6.5; type fixed -> revolute
- joint l_arm_grip: limit lower=0.0 upper=1.13446401394 effort=1000 velocity=6.5 -> lower=0.0 upper=1.1344640139444444 effort=1000 velocity=6.5; origin xyz=0.0877 0.0583 0.0 rpy=0 0 0.698131700889 -> xyz=0.0877 0.0583 0.0 rpy=0 0 0.6981317008888889
- joint l_arm_grip_1: limit lower=0.0 upper=1.13446401394 effort=1000 velocity=6.5 -> lower=0.0 upper=1.1344640139444444 effort=1000 velocity=6.5; origin xyz=0.0877 0.0317 0.0 rpy=0 0 -0.698131700889 -> xyz=0.0877 0.0317 0.0 rpy=0 0 -0.6981317008888889
- joint l_arm_wr_p: limit lower=-1.4137166943 upper=1.4137166943 effort=1000 velocity=6.5 -> lower=-1.4137166943000001 upper=1.4137166943000001 effort=1000 velocity=6.5
- joint l_arm_wr_r: limit lower=-2.8274333886 upper=2.8274333886 effort=1000 velocity=6.5 -> lower=-2.8274333886000003 upper=2.8274333886000003 effort=1000 velocity=6.5
- joint l_arm_wr_y: limit lower=-1.4137166943 upper=1.4137166943 effort=1000 velocity=6.5 -> lower=-1.4137166943000001 upper=1.4137166943000001 effort=1000 velocity=6.5
- joint l_leg_an_p: limit lower=-1.4137166943 upper=1.4137166943 effort=1000 velocity=6.5 -> lower=-1.4137166943000001 upper=1.4137166943000001 effort=1000 velocity=6.5
- joint l_leg_an_r: limit lower=-1.570796327 upper=1.2566370616 effort=1000 velocity=6.5 -> lower=-1.570796327 upper=1.2566370616000002 effort=1000 velocity=6.5
- joint l_leg_hip_p: limit lower=-1.2566370616 upper=1.2566370616 effort=1000 velocity=6.5 -> lower=-1.2566370616000002 upper=1.2566370616000002 effort=1000 velocity=6.5
- joint l_leg_hip_r: limit lower=-0.6283185308 upper=0.9424777962 effort=1000 velocity=6.5 -> lower=-0.6283185308000001 upper=0.9424777961999999 effort=1000 velocity=6.5
- joint l_leg_hip_y: limit lower=-1.4137166943 upper=1.4137166943 effort=1000 velocity=6.5 -> lower=-1.4137166943000001 upper=1.4137166943000001 effort=1000 velocity=6.5
- joint l_leg_kn_p: limit lower=-0.3141592654 upper=2.1991148578 effort=1000 velocity=6.5 -> lower=-0.31415926540000005 upper=2.1991148577999997 effort=1000 velocity=6.5
- joint r_arm_el_y: limit lower=-1.2566370616 upper=1.2566370616 effort=1000 velocity=6.5 -> lower=-1.2566370616000002 upper=1.2566370616000002 effort=1000 velocity=6.5
- joint r_arm_grip: limit lower=0.0 upper=1.13446401394 effort=1000 velocity=6.5 -> lower=0.0 upper=1.1344640139444444 effort=1000 velocity=6.5; origin xyz=0.0877 -0.0583 0.0 rpy=0 0 -0.698131700889 -> xyz=0.0877 -0.0583 0.0 rpy=0 0 -0.6981317008888889
- joint r_arm_grip_1: limit lower=0.0 upper=1.13446401394 effort=1000 velocity=6.5 -> lower=0.0 upper=1.1344640139444444 effort=1000 velocity=6.5; origin xyz=0.0877 -0.0317 0.0 rpy=0 0 0.698131700889 -> xyz=0.0877 -0.0317 0.0 rpy=0 0 0.6981317008888889
- joint r_arm_wr_p: limit lower=-1.4137166943 upper=1.4137166943 effort=1000 velocity=6.5 -> lower=-1.4137166943000001 upper=1.4137166943000001 effort=1000 velocity=6.5
- joint r_arm_wr_r: limit lower=-2.8274333886 upper=2.8274333886 effort=1000 velocity=6.5 -> lower=-2.8274333886000003 upper=2.8274333886000003 effort=1000 velocity=6.5
- joint r_arm_wr_y: limit lower=-1.4137166943 upper=1.4137166943 effort=1000 velocity=6.5 -> lower=-1.4137166943000001 upper=1.4137166943000001 effort=1000 velocity=6.5
- joint r_leg_an_p: limit lower=-1.4137166943 upper=1.4137166943 effort=1000 velocity=6.5 -> lower=-1.4137166943000001 upper=1.4137166943000001 effort=1000 velocity=6.5
- joint r_leg_an_r: limit lower=-1.4137166943 upper=1.4137166943 effort=1000 velocity=6.5 -> lower=-1.4137166943000001 upper=1.4137166943000001 effort=1000 velocity=6.5
- joint r_leg_hip_p: limit lower=-1.2566370616 upper=1.2566370616 effort=1000 velocity=6.5 -> lower=-1.2566370616000002 upper=1.2566370616000002 effort=1000 velocity=6.5
- joint r_leg_hip_r: limit lower=-0.9424777962 upper=0.6283185308 effort=1000 velocity=6.5 -> lower=-0.9424777961999999 upper=0.6283185308000001 effort=1000 velocity=6.5
- joint r_leg_hip_y: limit lower=-1.4137166943 upper=1.4137166943 effort=1000 velocity=6.5 -> lower=-1.4137166943000001 upper=1.4137166943000001 effort=1000 velocity=6.5
- joint r_leg_kn_p: limit lower=-2.1991148578 upper=0.3141592654 effort=1000 velocity=6.5 -> lower=-2.1991148577999997 upper=0.31415926540000005 effort=1000 velocity=6.5
- joint thormang3_fixed_gogoro: axis (none) -> 0 0 1; limit (none) -> lower=0.0 upper=0.0 effort=1000 velocity=6.5; type fixed -> revolute
- joint torso_y: limit lower=-1.8849555924 upper=1.8849555924 effort=1000 velocity=6.5 -> lower=-1.8849555923999999 upper=1.8849555923999999 effort=1000 velocity=6.5

Commit message: fixing the arms problem when scooter rotate

File: assets/urdf/thormang3/urdf/all.urdf (robot description, URDF)
Before this commit: robot gogoro_and_thormang3, 55 links, 54 joints
Links:
- removed link feet_visual
- removed link l_arm_end_link
- removed link r_arm_end_link
Joints:
- removed joint l_arm_end
- removed joint r_arm_end
- removed joint rigid4
